File: shunt_regulator/shunt_regulator.kicad_sch (KiCad schematic)
At the start: 15 parts

Commit message: Finished design
Parts:
- removed R? (x4): ?, symbol Device:R
- removed U?: LM393, symbol Comparator:LM393
- added C4: 1u, Diode_SMD:D_0805_2012Metric, symbol Device:C
- added C5, C6: 100n, Diode_SMD:D_0805_2012Metric, symbol Device:C
- added C7, C8: 47u, Capacitor_SMD:CP_Elec_10x10, symbol Device:C_Polarized
- added D3: LED, LED_SMD:LED_0805_2012Metric, symbol Device:LED
- added F1, F2: 500 mA, Fuse:Fuse_2920_7451Metric, symbol Device:Polyfuse
- added J1: Screw_Terminal_01x03, shunt_regulator_footprints:Owon SPE terminals, symbol Connector:Screw_Terminal_01x03
- added Q1, Q2: BC846B, Package_TO_SOT_SMD:SOT-23, symbol Transistor_BJT:BC846
- added Q3: BC856B, Package_TO_SOT_SMD:SOT-23, symbol Transistor_BJT:BC856
- added Q4: 30N06, Package_TO_SOT_SMD:TO-252-2, symbol Device:Q_NMOS_GDS
- added R1, R2, R37: 22k, Resistor_SMD:R_0805_2012Metric, symbol Device:R
- added R10, R9: 47k, Resistor_SMD:R_0805_2012Metric, symbol Device:R
- added R11, R6: 1k, Resistor_SMD:R_0805_2012Metric, symbol Device:R
- added R12, R13, R14, R15, R16, R17, R18, R19, R20, R21, R22, R23, R24, R25, R26, R27, R28, R29, R30, R31, R32, R33, R34, R35, R36: 100, Resistor_SMD:R_1210_3225Metric, symbol Device:R
- added R5, R7, R8: 10k, Resistor_SMD:R_0805_2012Metric, symbol Device:R
- added RV1: 100k, Potentiometer_THT:Potentiometer_Bourns_3296W_Vertical, symbol Device:R_Potentiometer
- added unit 2 of U2
- R3: renamed from R?; footprint (none) -> Resistor_SMD:R_0805_2012Metric; LCSC (none) -> C17572
- R4: renamed from R?; footprint (none) -> Resistor_SMD:R_0805_2012Metric; LCSC (none) -> C18359
- U2: renamed from U?; footprint (none) -> Package_SO:SOIC-8_3.9x4.9mm_P1.27mm; LCSC (none) -> C7955
- gave numbers to parts that had none: 7
Connections:
- net +VDC: now also C5.1, C6.1, C7.1, C8.1, F1.1, F2.1, J1.3 (Pin_3), Q1.3 (C), R1.2
- net GND: now also C4.2, C5.2, C6.2, C7.2, C8.2, J1.1 (Pin_1), Q3.2 (E), Q4.3 (S), R2.1, R5.1, R8.1
- net VCC: now also C4.1, Q2.3 (C), R10.2, R37.2, R7.1
- net at U2.2 (-): now also R7.2, R8.2, U2.6 (-)
- net at U2.1: now also R10.1, R11.1, R9.2
- net at U2.3 (+): now also R6.2, R9.1
- new net: R1.1, RV1.1, RV1.2
- new net: Q2.2 (E), Q3.3 (C), R12.1
- new net: Q4.1 (G), R12.2
- new net: F1.2, R13.2, R14.2, R15.2, R16.2, R17.2, R18.2, R25.2, R26.2, R27.2, R28.2, R29.2, R30.2
- new net: Q4.2 (D), R13.1, R14.1, R15.1, R16.1, R17.1, R18.1, R19.1, R20.1, R21.1, R22.1, R23.1, R24.1, R25.1, R26.1, R27.1, R28.1, R29.1, R30.1, R31.1, R32.1, R33.1, R34.1, R35.1, R36.1
- new net: Q1.1 (B), R2.2, RV1.3, U2.5 (+)
- new net: Q1.2 (E), R5.2, R6.1
- new net: F2.2, R19.2, R20.2, R21.2, R22.2, R23.2, R24.2, R31.2, R32.2, R33.2, R34.2, R35.2, R36.2
- new net: D3.1 (K), U2.7
- new net: D3.2 (A), R37.1
- new net: Q2.1 (B), Q3.1 (B), R11.2
- no-connect marks 0 -> 1
Other:
- moved on the sheet: U2A

Commit message: Changed the power resistor footprint from 1210 to 2512
Parts:
- R12, R13, R14, R15, R16, R17, R18, R19, R20, R21, R22, R23, R24, R25, R26, R27, R28, R29, R30, R31, R32, R33, R34, R35, R36: footprint Resistor_SMD:R_1210_3225Metric -> Resistor_SMD:R_2512_6332Metric
- R2: LCSC (none) -> C17560

Commit message: Fixed a push-pull transistor that was the wrong way around
Connections:
- net GND: now also Q3.3 (C); no longer Q3.2 (E)
- net at Q2.2 (E), R12.1: now also Q3.2 (E); no longer Q3.3 (C)
Changed lines of the file:
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@@
     (pin "2")
   )
-  (symbol (lib_id "Transistor_BJT:BC856") (at 134.62 144.78 0) (unit 1)
+  (symbol (lib_id "Transistor_BJT:BC856") (at 134.62 144.78 0) (mirror x) (unit 1)
     (in_bom yes) (on_board yes) (fields_autoplaced)
-    (property "Reference" "Q3" (id 0) (at 139.7 143.5099 0)
+    (property "Reference" "Q3" (id 0) (at 140.335 143.5099 0)
       (effects (font (size 1.27 1.27)) (justify left))
     )
-    (property "Value" "BC856B" (id 1) (at 139.7 146.0499 0)
+    (property "Value" "BC856B" (id 1) (at 140.335 146.0499 0)
       (effects (font (size 1.27 1.27)) (justify left))
     )
-    (property "Footprint" "Package_TO_SOT_SMD:SOT-23" (id 2) (at 139.7 146.685 0)
+    (property "Footprint" "Package_TO_SOT_SMD:SOT-23" (id 2) (at 139.7 142.875 0)
       (effects (font (size 1.27 1.27) italic) (justify left) hide)
     )

Commit message: Flipped input of LED comperator
Connections:
- net at R7.2, R8.2, U2.2 (-): now also U2.5 (+); no longer U2.6 (-)
- net at Q1.1 (B), R2.2, RV1.3: now also U2.6 (-); no longer U2.5 (+)
Changed lines of the file:
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@@
     (pin "2")
   )
-  (symbol (lib_id "Comparator:LM393") (at 107.95 175.26 0) (mirror x) (unit 2)
+  (symbol (lib_id "Comparator:LM393") (at 107.95 175.26 0) (unit 2)
     (in_bom yes) (on_board yes) (fields_autoplaced)
     (property "Reference" "U2" (id 0) (at 107.95 165.1 0))

Commit message: Changed the LCSC number of the 10k resistors
Parts:
- R5, R7, R8: LCSC C17724 -> C17414
Changed lines of the file:
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@@
       (effects (font (size 1.27 1.27)) hide)
     )
-    (property "LCSC" "C17724" (id 4) (at 92.71 146.05 90)
+    (property "LCSC" "C17414" (id 4) (at 92.71 146.05 90)
       (effects (font (size 1.27 1.27)) hide)
     )
@@
       (effects (font (size 1.27 1.27)) hide)
     )
-    (property "LCSC" "C17724" (id 4) (at 71.12 124.46 90)
+    (property "LCSC" "C17414" (id 4) (at 71.12 124.46 90)
       (effects (font (size 1.27 1.27)) hide)
     )
@@
       (effects (font (size 1.27 1.27)) hide)
     )
-    (property "LCSC" "C17724" (id 4) (at 86.36 139.7 90)
-      (effects (font (size 1.27 1.27)) hide)
-    )
+    (property "LCSC" "C17414" (id 4) (at 86.36 139.7 90)
+      (effects (font (size 1.27 1.27)) hide)
+    )
